File: reworked/frankless/frankless.kicad_pcb (KiCad board)
At the start: 4 copper layers, 32 x 74 mm, 116 parts, among them J1 GPIO, J10 BAT 3V, J2 DEBUG, J3 1040310811, J4 SS-52100-004, J5 USB4215-03-A, J6 HC-HDMI0019T-1A, J7 PJ-320D, J8 UART, U1 TS3USB221RSER, U10 DS3231MZ+TRL, U11 CH334R, U2 USBLC6-2SC6, U3 AMS1117-3.3, U5 APS6404L-3SQR-SN, U6 W25Q128JVS, U7 RP2350, U8 TDA1387T, U9 LM358, Y1 ASE-12MHz, Y2 12Mhz, Y3 ASE-12MHz

Commit message: A bit of clean up for things that don't make sense with the new layout yet
Parts:
- added G***: LOGO, Logo:Logo-15mm, B.Cu at (198.6, 111.6)
Other:
- board text added: "${NAME} Rev ${VERSION}"
- board text added: "Frankless Frank KiCad files https://github.com/arlaneenalra/pi-pico-boards/ tree/main/reworked/frankless Cloned from the MicroFrank Original https://frank.rh1.tech/hardware/microfrank Released under GPL V3"
- board text removed: "Frankless Frank KiCad https://github.com/arlaneenalra/pi-pico-boards Cloned from the MicroFrank Original https://frank.rh1.tech/hardware/microfrank"

Commit message: Patch a few minor issues.
Connections:
- net /RP2350A/GPI027/ADC1 renamed /RP2350A/GPIO27/ADC1
- C39 pad 2: +3V3 -> Net-(U11-VDD33_{LDO})
- C40 pad 2: +3V3 -> Net-(U11-VDD33_{LDO})
- U11 pad 13: +3V3 -> Net-(U11-VDD33_{LDO})
- U7 pad 3: /Micro SD/DAT0 -> /Micro SD/CDDAT3
- U7 pad 7: /Micro SD/CDDAT3 -> /Micro SD/DAT0
Routing:
- net Net-(U11-VDD33_{LDO}): track 0.00 -> 3.46 mm, vias 0 -> 1
- net +3V3: track 69.3 -> 65.8 mm, vias 25 -> 24
- net /Micro SD/CDDAT3: track 15.3 -> 18.0 mm, vias 0 -> 4
- net /Micro SD/DAT0: track 13.8 -> 14.5 mm

Commit message: More cleanup.
Parts:
- added C44: 10uf, Capacitor_SMD:C_0402_1005Metric, B.Cu at (196.1, 111.5)
- added R36: 10K, Resistor_SMD:R_0402_1005Metric, B.Cu at (198.0, 109.0)
- added R37: 10K, Resistor_SMD:R_0402_1005Metric, B.Cu at (193.2, 110.7)
- added R38: 10K, Resistor_SMD:R_0402_1005Metric, B.Cu at (196.2, 107.4)
- added R39: 10K, Resistor_SMD:R_0402_1005Metric, B.Cu at (198.5, 106.2)
- added R40: 10K, Resistor_SMD:R_0402_1005Metric, B.Cu at (192.7, 104.1)
- R34: value 4.7k -> 10K
- moved R34 17.2 mm to (193.2, 114.0)
Connections:
- R34 pad 2: /Real Time Clock/32KHZ -> /Micro SD/DAT2
- U10 pad 1: /Real Time Clock/32KHZ -> unconnected-(U10-32KHZ-Pad1)
Routing:
- net +3V3: track 65.8 -> 71.8 mm, vias 24 -> 30
- net /Micro SD/DAT1: track 0.00 -> 2.31 mm, vias 0 -> 1
- net /Real Time Clock/32KHZ: track 1.75 -> 0.00 mm
- net /Micro SD/DAT2: track 0.00 -> 1.65 mm, vias 0 -> 1
- net /Micro SD/CDDAT3: track 18.0 -> 19.4 mm
- net /Micro SD/CLK: track 14.4 -> 15.5 mm, vias 0 -> 1
- net /Micro SD/DAT0: track 14.5 -> 15.5 mm
- net /Micro SD/CMD: track 15.1 -> 15.8 mm, vias 0 -> 1
- net GND: vias 69 -> 72
