File: reworked/frankless/frankless.kicad_pcb (KiCad board)
At the start: 4 copper layers, 32 x 74 mm, 123 parts, among them J1 GPIO, J10 BAT 3V, J2 DEBUG, J3 1040310811, J4 SS-52100-004, J5 USB4215-03-A, J6 HC-HDMI0019T-1A, J7 PJ-320D, J8 UART, U1 TS3USB221RSER, U10 DS3231MZ+TRL, U11 CH334R, U2 USBLC6-2SC6, U3 AMS1117-3.3, U5 APS6404L-3SQR-SN, U6 W25Q128JVS, U7 RP2350, U8 TDA1387T, U9 LM358, Y1 ASE-12MHz, Y2 12Mhz, Y3 ASE-12MHz

Commit message: Fixing bad footprint matches.
Parts:
- removed J4: SS-52100-004, MicroFRANK:USB_A_Stacked
- removed J5: USB4215-03-A, MicroFRANK:USB_C_Receptacle
- added USB1: AF SS-JB17.6, EasyEDA_Lib:USB-A-TH_AF-SS-JB17.6, F.Cu at (206.5, 68.5)
- added USBC1: USB4215-03-A, EasyEDA_Lib:USB-C_SMD-TYPE-C-31-M-12_1, F.Cu at (194.5, 86.5)
- L1: value 330R -> 120R
- R35: value 4.7k -> 4.7K
- moved R7 3.53 mm to (199.4, 84.7)
- moved R6 3.33 mm to (199.4, 87.9)
Connections:
- J3 pad 1: /Micro SD/DAT2 -> unconnected-(J3-DAT2-Pad1)
- J3 pad 10: /Micro SD/DET_A -> unconnected-(J3-DET_A-Pad10)
- J3 pad 8: /Micro SD/DAT1 -> unconnected-(J3-DAT1-Pad8)
- J3 pad 9: /Micro SD/DET_B -> unconnected-(J3-DET_B-Pad9)
- R34 pad 2: /Micro SD/DAT2 -> unconnected-(J3-DAT2-Pad1)
- R40 pad 2: /Micro SD/DAT1 -> unconnected-(J3-DAT1-Pad8)
Routing:
- net unconnected-(J3-DAT1-Pad8): track 0.00 -> 2.31 mm, vias 0 -> 1
- net /Micro SD/DAT1: track 2.31 -> 0.00 mm, vias 1 -> 0
- net unconnected-(J3-DAT2-Pad1): track 0.00 -> 1.65 mm, vias 0 -> 1
- net /Micro SD/DAT2: track 1.65 -> 0.00 mm, vias 1 -> 0
- net Net-(R1-Pad2): track 9.37 -> 9.92 mm, vias 1 -> 0
- net Net-(R8-Pad1): track 18.8 -> 18.3 mm
- net Net-(R5-Pad2): track 4.24 -> 4.59 mm, vias 0 -> 1
- net Net-(R4-Pad2): track 5.44 -> 5.68 mm, vias 1 -> 0
- net Net-(R3-Pad2): track 7.66 -> 7.87 mm, vias 0 -> 1
- net GND: vias 72 -> 69

Commit message: Fixing bad footprint matches.
Parts:
- removed USBC1: USB4215-03-A, EasyEDA_Lib:USB-C_SMD-TYPE-C-31-M-12_1
- added USB2: USB4215-03-A, EasyEDA_Lib:USB-C-SMD_GT-USB-7010B, F.Cu at (194.5, 86.3)
- moved R8 0.45 mm to (193.6, 86.6)
Routing:
- net Net-(USB2-Dp1): track 3.74 -> 4.92 mm
- net /Power/VBUS_IN: track 17.9 -> 17.0 mm
- net Net-(USB2-Dn1): track 4.72 -> 3.84 mm
- net Net-(R8-Pad1): track 18.3 -> 19.2 mm
- net GND: vias 69 -> 67

Commit message: More PCB layout clean ups.
Parts:
- added C7: 10uf, Capacitor_SMD:C_0603_1608Metric, B.Cu at (197.5, 95.5)
- C4: value 22uf -> 10uf
Connections:
- J3 pad 1: unconnected-(J3-DAT2-Pad1) -> Net-(J3-DAT2)
- J3 pad 8: unconnected-(J3-DAT1-Pad8) -> Net-(J3-DAT1)
- R34 pad 2: unconnected-(J3-DAT2-Pad1) -> Net-(J3-DAT2)
- R40 pad 2: unconnected-(J3-DAT1-Pad8) -> Net-(J3-DAT1)
Routing:
- net unconnected-(J3-DAT1-Pad8): track 2.31 -> 0.00 mm, vias 1 -> 0
- net Net-(J3-DAT1): track 0.00 -> 2.31 mm, vias 0 -> 1
- net unconnected-(J3-DAT2-Pad1): track 1.65 -> 0.00 mm, vias 1 -> 0
- net Net-(J3-DAT2): track 0.00 -> 1.65 mm, vias 0 -> 1

Commit message: Fix reset and boot button.
Parts:
- turned S3 to 180 degrees
Connections:
- S3 pad 1: GND -> /RP Reset/C1
- S3 pad 4: /RP Reset/C1 -> GND
- S4 pad 1: GND -> /RP2350A/~{USB_BOOT}
- S4 pad 4: /RP2350A/~{USB_BOOT} -> GND
Routing:
- net /RP2350A/~{USB_BOOT}: track 12.0 -> 13.1 mm
- net /RP Reset/C1: track 35.1 -> 34.4 mm
