File: reworked/frankless/RealTimeClock.kicad_sch (KiCad schematic)
At the start: 7 parts, among them J10 BAT 3V, U10 DS3231MZ+TRL

Commit message: More cleanup.
Parts:
- removed R34: 4.7k, Resistor_SMD:R_0402_1005Metric, symbol MicroFRANK:R
Connections:
- net 32KHZ: no longer names the net of U10.1 (32KHZ)
- no-connect marks 1 -> 3

Commit message: Fixing bad footprint matches.
Parts:
- R35: value 4.7k -> 4.7K
