File: reworked/frankless/audio.kicad_sch (KiCad schematic)
At the start: 1 part, among them J7 PJ-320D

Commit message: Fixing bad footprint matches.
Parts:
- J7: AliExpress https://jlcpcb.com/partdetail/Korean_HropartsElec-PJ_320DB5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 -> https://jlcpcb.com/partdetail/SHOUHAN-PJ320D/C431535; LCSC Part # C707225 -> C431535
Changed lines of the file:
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@@
 			)
 		)
-		(property "AliExpress" "https://jlcpcb.com/partdetail/Korean_HropartsElec-PJ_320DB5A/C707225"
+		(property "AliExpress" "https://jlcpcb.com/partdetail/SHOUHAN-PJ320D/C431535"
 			(at 187.96 99.06 0)
 			(hide yes)
@@
 			)
 		)
-		(property "LCSC Part #" "C707225"
+		(property "LCSC Part #" "C431535"
 			(at 187.96 99.06 0)
 			(hide yes)
@@
 			(at 187.96 99.06 0)
 			(hide yes)
+			(show_name no)
+			(do_not_autoplace no)
+			(effects
+				(font
+					(size 1.27 1.27)
+				)
+			)
+		)
+		(property "LCSC Part Name" ""
+			(at 187.96 99.06 0)
+			(hide yes)
+			(show_name no)
+			(do_not_autoplace no)
+			(effects
+				(font
+					(size 1.27 1.27)
+				)
+			)
+		)
+		(property "Manufacturer Part" ""
+			(at 187.96 99.06 0)
+			(hide yes)
+			(show_name no)
+			(do_not_autoplace no)
+			(effects
+				(font
+					(size 1.27 1.27)
+				)
+			)
+		)
+		(property "Supplier" ""
+			(at 187.96 99.06 0)
+			(hide yes)
+			(show_name no)
+			(do_not_autoplace no)
+			(effects
+				(font
+					(size 1.27 1.27)
+				)
+			)
+		)
+		(property "Supplier Part" ""
+			(at 187.96 99.06 0)
+			(hide yes)
+			(show_name no)
+			(do_not_autoplace no)
+			(effects
+				(font
+					(size 1.27 1.27)
+				)
+			)
+		)
+		(property "LCSC" ""
+			(at 187.96 99.06 0)
+			(hide yes)
