File: reworked/frankless/frankless.kicad_sch (KiCad schematic)
At the start: 8 parts, among them J1 GPIO, J2 DEBUG, J8 UART

Commit message: A bit of clean up for things that don't make sense with the new layout yet
Other:
- company: Mikhail Matveev -> Chris Salch
Changed lines of the file:
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@@
 		(date "${DATE}")
 		(rev "${VERSION}")
-		(company "Mikhail Matveev")
-		(comment 1 "https://github.com/rh1tech/frank")
+		(company "Chris Salch")
+		(comment 1 "https://github.com/arlaneenalra/pi-pico-boards/tree/main/reworked/frankless")
+		(comment 2 "Orignal By")
+		(comment 3 "Mikhail Matveev")
+		(comment 4 "https://github.com/rh1tech/frank")
 	)
 	(junction

Commit message: Patch a few minor issues.
Connections:
- net RP2350A/GPI027/ADC1 renamed RP2350A/GPIO27/ADC1
- no-connect marks 0 -> 1
Other:
- sheet RP2350A ports: added GPIO27/ADC1; removed 32KHZ, GPI027/ADC1
Changed lines of the file:
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@@
 		(color 0 0 0 0)
 	)
+	(no_connect
+		(at 102.87 82.55)
+	)
 	(wire
 		(pts
@@
 		(pts
 			(xy 107.95 115.57) (xy 123.19 115.57)
-		)
-		(stroke
-			(width 0)
-			(type default)
-		)
-	)
-	(wire
-		(pts
-			(xy 102.87 82.55) (xy 123.19 82.55)
 		)
 		(stroke
@@
 			)
 		)
-		(pin "32KHZ" input
-			(at 123.19 82.55 180)
-			(effects
-				(font
-					(size 1.27 1.27)
-				)
-				(justify left)
-			)
-		)
-		(pin "GPI027{slash}ADC1" tri_state
+		(pin "GPIO27{slash}ADC1" tri_state
 			(at 123.19 118.11 180)
 			(effects

Commit message: More cleanup.
Connections:
- no-connect marks 1 -> 0
Other:
- sheet Real Time Clock ports: added none; removed 32KHZ
Changed lines of the file:
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@@
 		(color 0 0 0 0)
 	)
-	(no_connect
-		(at 102.87 82.55)
-	)
 	(wire
 		(pts
@@
 			(effects
 				(font
-					(size 1.27 1.27)
-				)
-				(justify right)
-			)
-		)
-		(pin "32KHZ" input
-			(at 102.87 82.55 0)
-			(effects
-				(font
