File: reworked/frankless/rp2350a.kicad_sch (KiCad schematic)
At the start: 31 parts, among them U5 APS6404L-3SQR-SN, U6 W25Q128JVS, U7 RP2350, Y1 ASE-12MHz

Commit message: Patch a few minor issues.
Connections:
- net SD_CDDAT3: now also U7.3 (GPIO1); no longer U7.7 (GPIO4)
- net SD_DAT0: now also U7.7 (GPIO4); no longer U7.3 (GPIO1)
- net GPI027/ADC1 renamed GPIO27/ADC1
Changed lines of the file:
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@@
 		)
 	)
-	(hierarchical_label "SD_DAT0"
+	(hierarchical_label "SD_CDDAT3"
 		(shape input)
 		(at 227.33 74.93 0)
@@
 		)
 	)
-	(hierarchical_label "GPI027{slash}ADC1"
+	(hierarchical_label "GPIO27{slash}ADC1"
 		(shape tri_state)
 		(at 227.33 143.51 0)
@@
 		)
 	)
-	(hierarchical_label "SD_CDDAT3"
+	(hierarchical_label "SD_DAT0"
 		(shape input)
 		(at 227.33 82.55 0)

Commit message: Fix a few parts.
Parts:
- R16, R17: LCSC Part # C25905 -> C11702
Changed lines of the file:
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@@
 			)
 		)
-		(property "LCSC Part #" "C25905"
+		(property "LCSC Part #" "C11702"
 			(at 144.78 184.15 90)
 			(hide yes)
@@
 			)
 		)
-		(property "LCSC Part #" "C25905"
+		(property "LCSC Part #" "C11702"
 			(at 127 83.82 90)
 			(hide yes)
