File: reworked/frankless/sd.kicad_sch (KiCad schematic)
At the start: 2 parts, among them J3 1040310811

Commit message: More cleanup.
Parts:
- added C44: 10uf, Capacitor_SMD:C_0402_1005Metric, symbol MicroFRANK:C
- added R34, R36, R37, R38, R39, R40: 10K, Resistor_SMD:R_0402_1005Metric, symbol MicroFRANK:R
Connections:
- net +3V3: now also C44.2, R34.1, R36.1, R37.1, R38.1, R39.1, R40.1
- net CDDAT3: now also R36.2
- net CLK: now also R38.2
- net CMD: now also R37.2
- net DAT0: now also R39.2
- net GND: now also C44.1
- net DAT1: no longer names the net of J3.8 (DAT1)
- net DAT1: now also R40.2
- net DAT2: no longer names the net of J3.1 (DAT2)
- net DAT2: now also R34.2
- net DET_A: no longer names the net of J3.10 (DET_A)
- net DET_B: no longer names the net of J3.9 (DET_B)
- no-connect marks 0 -> 4
Other:
- moved on the sheet: C37

Commit message: Fix a few parts.
Changed lines of the file:
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@@
+	(wire
+		(pts
+			(xy 182.88 109.22) (xy 177.8 109.22)
+		)
+		(stroke
+			(width 0)
+			(type default)
+		)
+	)
 	(wire
 		(pts
@@
 	(symbol
 		(lib_id "MicroFRANK:GND")
-		(at 177.8 109.22 0)
+		(at 182.88 109.22 0)
 		(unit 1)
 		(body_style 1)
@@
 		(fields_autoplaced yes)
 		(property "Reference" "#PWR01"
-			(at 177.8 115.57 0)
+			(at 182.88 115.57 0)
 			(hide yes)
 			(show_name no)
@@
 		)
 		(property "Value" "GND"
-			(at 177.8 114.3 0)
+			(at 182.88 114.3 0)
 			(show_name no)
 			(do_not_autoplace no)
@@
 		)
 		(property "Footprint" ""
-			(at 177.8 109.22 0)
+			(at 182.88 109.22 0)
 			(hide yes)
 			(show_name no)
@@
 		)
 		(property "Datasheet" ""
-			(at 177.8 109.22 0)
+			(at 182.88 109.22 0)
 			(hide yes)
 			(show_name no)
@@
 		)
 		(property "Description" "Power symbol creates a global label with name \"GND\" , ground"
-			(at 177.8 109.22 0)
-			(hide yes)
-			(show_name no)
+			(at 182.88 109.22 0)
+			(hide yes)
+			(show_name no)

Commit message: More PCB layout clean ups.
Connections:
- no-connect marks 4 -> 2
Changed lines of the file:
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@@
-	)
-	(junction
-		(at 129.54 86.36)
-		(diameter 0)
-		(color 0 0 0 0)
 	)
 	(junction
@@
 		(color 0 0 0 0)
 	)
-	(junction
-		(at 68.58 104.14)
-		(diameter 0)
-		(color 0 0 0 0)
-	)
-	(no_connect
-		(at 127 86.36)
-	)
 	(no_connect
 		(at 127 109.22)
@@
 	(no_connect
 		(at 127 106.68)
-	)
-	(no_connect
-		(at 66.04 104.14)
 	)
 	(wire
@@
 		(pts
 			(xy 80.01 101.6) (xy 134.62 101.6)
-		)
-		(stroke
-			(width 0)
-			(type default)
-		)
-	)
-	(wire
-		(pts
-			(xy 66.04 104.14) (xy 68.58 104.14)
 		)
 		(stroke
@@
 		)
 		(stroke
-			(width 0)
-			(type default)
-		)
-	)
-	(wire
-		(pts
-			(xy 127 86.36) (xy 129.54 86.36)
-		)
-		(stroke
